File: Wham-Link.kicad_pcb (KiCad board)
At the start: 4 copper layers, 70 x 30 mm, 45 parts, among them J2 Conn_02x05_Counter_Clockwise, J3 Conn_01x09_Pin, SW2 SKRPACE010, SW3 SKRPACE010, U1 LAN8720A-CP-TR, U2 AMS1117-3.3, U3 CH340C, U4 ESP32-WROOM-32UE, X1 ECS-2520MV-250-CN-TR

Commit message: Schematic and layout updates
Parts:
- moved C2 3.76 mm to (146.9, 107.6), turned to 45 degrees
- moved R15 3.35 mm to (153.4, 110.5), turned to 180 degrees
- moved C10 1.00 mm to (132.2, 102.7), turned to 180 degrees
Routing:
- net +3V3: track 29.1 -> 129.8 mm, vias 0 -> 4
- net +5V: track 12.8 -> 60.8 mm, vias 0 -> 2
- net BOOT: track 55.5 -> 56.6 mm
- net IO23: track 45.8 -> 46.4 mm
